Commit message: map on rviz but costmap not working

File: install/sam_bot_description/share/sam_bot_description/src/description/sam_bot_description.urdf (robot description, URDF)
Before this commit: robot sam_bot, 3 links, 2 joints
Links:
- added link camera_depth_frame
- added link camera_link, mass 0.035; collision box size=0.015 0.130 0.022; visual box size=0.015 0.130 0.022
- added link imu_link; collision box size=0.1 0.1 0.1; visual box size=0.1 0.1 0.1
- added link lidar_link, mass 0.125; collision cylinder length=0.055 radius=0.0508; visual cylinder length=0.055 radius=0.0508
Joints:
- added joint camera_depth_joint: type fixed, parent camera_link, child camera_depth_frame, origin xyz=0 0 0 rpy=${-pi/2} 0 ${-pi/2}
- added joint camera_joint: type fixed, parent base_link, child camera_link, origin xyz=0.215 0 0.05 rpy=0 0 0
- added joint imu_joint: type fixed, parent base_link, child imu_link, origin xyz=0 0 0.01
- added joint lidar_joint: type fixed, parent base_link, child lidar_link, origin xyz=0 0 0.12 rpy=0 0 0
