Commit message: Add files via upload

File: src/sam_bot_description/src/description/sam_bot_description.urdf (robot description, URDF)
Before this commit: robot sam_bot, 7 links, 6 joints
Links:
- link imu_link: geometry collision box size=0.1 0.1 0.1; visual box size=0.05 0.05 0.05
- link lidar_link: geometry collision cylinder length=0.055 radius=0.0508; visual cylinder length=0.0275 radius=0.0254
Joints:
- joint camera_joint: origin xyz=0.215 0 0.05 rpy=0 0 0 -> xyz=0.1075 0 0.025 rpy=0 0 0
- joint lidar_joint: origin xyz=0 0 0.12 rpy=0 0 0 -> xyz=0 0 0.06 rpy=0 0 0
